File: tone-bender-mk3.kicad_sch (KiCad schematic)
At the start: 47 parts, among them P1 IN, P2 GND, P3 -9V, P4 LED+, P5 GND, P6 GND, P7 OUT, P8 GND, Q1 Q_PNP_BCE, Q2 Q_PNP_BCE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

Commit message: donezo
exporting for quote now
Parts:
- removed C13, C14: 100n, Capacitor_SMD:C_0402_1005Metric_Pad0.74x0.62mm_HandSolder, symbol Device:C
- removed D1: D, symbol Device:D
- removed D2: LED, LED_THT:LED_D5.0mm, symbol Device:LED
- removed P4: LED+, BB_Pads:WirePad_22AWG, symbol BlackBox:WirePad_22AWG
- removed P5: GND, BB_Pads:WirePad_22AWG, symbol BlackBox:WirePad_22AWG
- removed Q1, Q2, Q3: Q_PNP_BCE, BlackBox:Transistor_Generic_TO-5, symbol Device:Q_PNP_BCE
- removed R13: 4.7k, BB_Resistors:R_Axial_DIN0207_L6.3mm_D2.5mm_P7.5mm_Horizontal, symbol Device:R_US
- removed RV1, RV2, RV3: 100k, Potentiometer_THT:Potentiometer_Alpha_RD901F-40-00D_Single_Vertical, symbol Device:R_Potentiometer_US
- removed RV4, RV5: 10k, symbol Device:R_Potentiometer_Trim
- added D4: 1N34A, BB_Diodes:D_DO-41_SOD81_P10.0mm_Horizontal, symbol #gplm:dio/DIO-0001-0001
- added Q1, Q2: PNP_Ge, BB_Transistor:TO-92L_Wide_EBC, symbol #gplm:xtr/XTR-0002-0001
- added Q3: PNP_Ge, BB_Transistor:TO-92L_Wide_EBC, symbol #gplm:xtr/XTR-0002-0003
- added RV1, RV2, RV3: B100k, BB_Potentiometers:Potentiometer_16MM, symbol #gplm:pot/POT-0002-0007
- added RV4, RV5: B20k, BB_Potentiometers:Potentiometer_Bourns_3362P_Vertical, symbol #gplm:pot/POT-0005-0005
- D1: renamed from D3; value 1N4001 -> 1N4001G-T; footprint Diode_THT:D_DO-41_SOD81_P10.16mm_Horizontal -> BB_Diodes:D_DO-41_SOD81_P7.5mm_Horizontal; symbol Diode:1N4001 -> #gplm:dio/DIO-0002-0001; Current (none) -> 1A; IPN (none) -> DIO-0002-0001; MPN (none) -> 1N4001G-T; Manufacturer (none) -> Diodes Incorporated; Voltage (none) -> 1V @ 1A
- R1, R11, R12, R3, R4, R6, R7, R8, R9: footprint Resistor_THT:R_Axial_DIN0207_L6.3mm_D2.5mm_P10.16mm_Horizontal -> BB_Resistors:R_Axial_DIN0207_L6.3mm_D2.5mm_P7.5mm_Horizontal
- R10: value 10k -> 4.7k; footprint Resistor_THT:R_Axial_DIN0207_L6.3mm_D2.5mm_P10.16mm_Horizontal -> BB_Resistors:R_Axial_DIN0207_L6.3mm_D2.5mm_P7.5mm_Horizontal
- R2: value 15k -> 10k; footprint Resistor_THT:R_Axial_DIN0207_L6.3mm_D2.5mm_P10.16mm_Horizontal -> BB_Resistors:R_Axial_DIN0207_L6.3mm_D2.5mm_P7.5mm_Horizontal
Connections:
- net VDD is gone; now on net -9V: C10.1, C3.2, D1.2 (A), R11.2, R14.2, R9.2
- net GND: now also D4.1 (K), Q3.1 (E), RV3.1
- net OUT: now also RV3.2
- net Q1_B: now also Q1.2 (B)
- net Q1_C: now also Q1.3 (C), Q2.3 (C)
- net Q1_C_AC: now also RV1.3
- net Q1_C_DIV: now also RV4.3
- net Q2_B: now also Q1.1 (E), Q2.2 (B)
- net Q2_E: now also Q2.1 (E)
- net Q3_B: now also D4.2 (A), Q3.2 (B), RV1.1, RV1.2
- net Q3_C: now also Q3.3 (C)
- net Q3_C_DIV: now also RV5.1, RV5.2
- net Q3_C_DIV_AC: now also RV2.1
- net TONE: now also RV2.2
- net TONE_DIV: now also RV3.3
- net TREB: now also RV2.3
- net at R2.2: now also RV5.3
- net +9V renamed -9V
- net -9V: now also RV4.1, RV4.2
